Commit message: 增加定位包

File: src/wcmodel/urdf/wheelchair_base.urdf (robot description, URDF)
Before this commit: robot wheelchair, 8 links, 7 joints
Joints:
- joint laser_joint: origin xyz=0 0 0.325 -> xyz=0.4 0.3 0.1

Commit message: 更新控制器逻辑;修改里程计主题

File: src/wcmodel/urdf/wheelchair_base.urdf (robot description, URDF)
Before this commit: robot wheelchair, 8 links, 7 joints
Links:
- link base_link: geometry collision box size=1.18 0.6 0.65; visual box size=1.18 0.6 0.65
- link left_small_wheel_link: geometry collision cylinder length=0.2 radius=0.12; visual cylinder length=0.04 radius=0.12
- link left_wheel_link: geometry collision cylinder length=0.2 radius=0.27; visual cylinder length=0.05 radius=0.27
- link right_small_wheel_link: geometry collision cylinder length=0.2 radius=0.12; visual cylinder length=0.04 radius=0.12
- link right_wheel_link: geometry collision cylinder length=0.2 radius=0.27; visual cylinder length=0.05 radius=0.27
Joints:
- joint laser_joint: origin xyz=0.4 0.3 0.1 -> xyz=0.0 0.2 0.1

Commit message: 修复bug

File: src/wcmodel/urdf/wheelchair_base.urdf (robot description, URDF)
Before this commit: robot wheelchair, 8 links, 7 joints
Joints:
- joint base_joint: child base_footprint -> base_link; origin xyz=0 0 -0.54 rpy=0 0 0 -> xyz=0 0 0.54 rpy=0 0 0; parent base_link -> base_footprint

Commit message: 更新wcmodel

File: src/wcmodel/urdf/wheelchair_base.urdf (robot description, URDF)
Before this commit: robot wheelchair, 8 links, 7 joints
Links:
- removed link left_small_wheel_link
- removed link left_wheel_link
- removed link right_small_wheel_link
- removed link right_wheel_link
- added link rabbit_link; visual mesh filename=package://wcmodel/meshes/rabbit.STL scale=${rabbit_scale} ${rabbit_scale*1.2} ${rabbit_scale}
- link base_link: geometry collision box size=${base_length} ${base_width} 0.3; visual mesh filename=package://wcmodel/meshes/robot_base.STL scale=1.0 1.0 1.0
Joints:
- removed joint left_small_wheel_joint
- removed joint left_wheel_joint
- removed joint right_small_wheel_joint
- removed joint right_wheel_joint
- added joint base_rabbit_joint: type fixed, parent base_link, child rabbit_link, origin xyz=-0.2 0 -0.08
- joint base_joint: origin xyz=0 0 0.54 rpy=0 0 0 -> xyz=0 0 ${(wheel_radius+wheel_zoff)} rpy=0 0 0
- joint imu_joint: origin xyz=0 0 0.30 -> xyz=0 0 0.01; parent base_link -> laser_link
- joint laser_joint: origin xyz=0.0 0.2 0.1 -> xyz=0.0 0.25 0.25

Commit message: 导航1.0问世

File: src/wcmodel/urdf/wheelchair_base.urdf (robot description, URDF)
Before this commit: robot wheelchair_base, 5 links, 4 joints
Joints:
- joint laser_joint: origin xyz=0.0 0.25 0.25 -> xyz=-0.25 0.25 0.25
