Commit message: 整理文件结构

File: src/wcmodel/urdf/gkchair01_base.urdf (robot description, URDF)
Before this commit: robot gk01, 4 links, 3 joints
Links:
- added link laser_ms200_link; visual cylinder length=0.02 radius=0.02
Joints:
- added joint laser_ms200_joint: type fixed, parent left_wheel_link, child laser_ms200_link, origin xyz=0.04 0.01 0.35
- joint laser_joint: origin xyz=0.37 -0.25 -0.16 -> xyz=0.075 0 ${s_wheel_radius+0.02}; parent base_link -> right_small_wheel_link
