Commit message: 增加新的模拟功能包

File: src/swc_nav_bringup/urdf/sentry_robot_real.xacro (robot description, xacro)
@@ -133,5 +133,5 @@
       <origin xyz="0.025 -0.0265 -0.025" rpy="${pi/2} 0 ${pi}"/>
       <geometry>
-        <mesh filename="package://pb_rm_simulation/meshes/mid360.stl" scale="0.001 0.001 0.001"/>
+        <mesh filename="package://pb_swc_simulation/meshes/mid360.stl" scale="0.001 0.001 0.001"/>
       </geometry>
       <material name="blue">

Commit message: 基于fastlio的导航测试成功

File: src/swc_nav_bringup/urdf/sentry_robot_real.xacro (robot description, xacro)
@@ -14,4 +14,10 @@
   <xacro:arg name="xyz" default="0.0 0.045 0.49" />
   <xacro:arg name="rpy" default="0 0 0" />
+  <link name="base_footprint" />
+  <joint name="base_joint" type="fixed">
+    <parent link="base_footprint" />
+    <child link="base_link" />
+    <origin xyz="0 0 0.05" rpy="0 0 0" />
+  </joint>
   <link name="base_link">
     <visual>
