Commit message: 文件结构优化

File: src/swc_nav_bringup/urdf/gkchair01_base.urdf (robot description, URDF)
Before this commit: robot wheelchair_base, 5 links, 4 joints
Links:
- removed link rabbit_link
- added link laser_ms200_link; visual cylinder length=0.02 radius=0.02
- link base_link: geometry collision box size=${base_length} ${base_width} 0.3; visual box size=${base_length} ${base_width} ${base_height}
Joints:
- removed joint base_rabbit_joint
- added joint laser_ms200_joint: type fixed, parent left_wheel_link, child laser_ms200_link, origin xyz=0.04 0.01 0.35
- joint laser_joint: origin xyz=-0.25 0.25 0.25 -> xyz=0.075 0 ${s_wheel_radius+0.02}; parent base_link -> right_small_wheel_link

File: src/swc_nav_bringup/urdf/wheelchair_base.urdf (robot description, URDF)
Before this commit: robot gk01, 5 links, 4 joints
Links:
- removed link laser_ms200_link
- added link rabbit_link; visual mesh filename=package://swc_nav_bringup/meshes/rabbit.STL scale=${rabbit_scale} ${rabbit_scale*1.2} ${rabbit_scale}
- link base_link: geometry collision box size=${base_length} ${base_width} 0.3; visual mesh filename=package://swc_nav_bringup/meshes/robot_base.STL scale=1.0 1.0 1.0
Joints:
- removed joint laser_ms200_joint
- added joint base_rabbit_joint: type fixed, parent base_link, child rabbit_link, origin xyz=-0.2 0 -0.08
- joint laser_joint: origin xyz=0.075 0 ${s_wheel_radius+0.02} -> xyz=-0.25 0.25 0.25; parent right_small_wheel_link -> base_link

Commit message: 暂存更改

File: src/swc_nav_bringup/urdf/gkchair01_base.urdf (robot description, URDF)
Before this commit: robot gk01, 5 links, 4 joints
Links:
- added link livox_frame; visual cylinder length=0.02 radius=0.02
Joints:
- added joint livox_frame_joint: type fixed, parent base_link, child livox_frame, origin xyz=0.44 ${base_width/2} ${-(wheel_radius+wheel_zoff)+s_wheel_radius*2 + 0.02}
- joint laser_joint: origin xyz=0.075 0 ${s_wheel_radius+0.02} -> xyz=0.44 ${-base_width/2} ${-(wheel_radius+wheel_zoff)+s_wheel_radius*2 + 0.02}; parent right_small_wheel_link -> base_link
- joint laser_ms200_joint: origin xyz=0.04 0.01 0.35 -> xyz=-0.285 0.305 0.125; parent left_wheel_link -> base_link

Commit message: 这个版本不乱转了，问题是走走停停

File: src/swc_nav_bringup/urdf/gkchair01_base.urdf (robot description, URDF)
Before this commit: robot gk01, 6 links, 5 joints
Links:
- added link drive_footprint
Joints:
- added joint drive_footprint_joint: type fixed, parent base_footprint, child drive_footprint, origin xyz=${-wheel_xoff} 0 0 rpy=0 0 0

Commit message: 调整urdf模型；调整局部代价地图参考系

File: src/swc_nav_bringup/urdf/gkchair01_base.urdf (robot description, URDF)
Before this commit: robot gk01, 7 links, 6 joints
Joints:
- joint base_joint: origin xyz=0 0 ${(wheel_radius+wheel_zoff)} rpy=0 0 0 -> xyz=0 0 ${base_link_high} rpy=0 0 0
- joint drive_footprint_joint: origin xyz=${-wheel_xoff} 0 0 rpy=0 0 0 -> xyz=${-wheel_xoff} 0 ${-base_link_high} rpy=0 0 0; parent base_footprint -> base_link
- joint laser_joint: origin xyz=0.44 ${-base_width/2} ${-(wheel_radius+wheel_zoff)+s_wheel_radius*2 + 0.02} -> xyz=${0.65-wheel_xoff} ${-s_wheel_ygap/2} ${-base_link_high+0.31}
- joint laser_ms200_joint: origin xyz=-0.285 0.305 0.125 -> xyz=${-wheel_xoff+0.1} ${wheel_ygap/2} ${-base_link_high + 0.53}
- joint livox_frame_joint: origin xyz=0.44 ${base_width/2} ${-(wheel_radius+wheel_zoff)+s_wheel_radius*2 + 0.02} -> xyz=${0.65-wheel_xoff} ${s_wheel_ygap/2} ${-base_link_high+ 0.31}

Commit message: 修正模型

File: src/swc_nav_bringup/urdf/gkchair01_base.urdf (robot description, URDF)
Before this commit: robot gk01, 7 links, 6 joints
Joints:
- joint laser_joint: origin xyz=${0.65-wheel_xoff} ${-s_wheel_ygap/2} ${-base_link_high+0.31} -> xyz=${0.61-wheel_xoff} ${-s_wheel_ygap/2} ${-base_link_high+0.335}
- joint laser_ms200_joint: origin xyz=${-wheel_xoff+0.1} ${wheel_ygap/2} ${-base_link_high + 0.53} -> xyz=${-wheel_xoff-0.1} 0 ${-base_link_high + 0.2}
- joint livox_frame_joint: origin xyz=${0.65-wheel_xoff} ${s_wheel_ygap/2} ${-base_link_high+ 0.31} -> xyz=${0.63-wheel_xoff} ${s_wheel_ygap/2} ${-base_link_high+ 0.345}

Commit message: 修改base_footprint未知

File: src/swc_nav_bringup/urdf/gkchair01_base.urdf (robot description, URDF)
Before this commit: robot gk01, 7 links, 6 joints
Links:
- removed link drive_footprint
- link base_link: geometry collision box size=${base_length} ${base_width} ${base_height}; visual box size=${base_length} ${base_width} ${base_height}
Joints:
- removed joint drive_footprint_joint
- joint base_joint: origin xyz=0 0 ${base_link_high} rpy=0 0 0 -> xyz=${wheel_xoff} 0 ${base_link_high} rpy=0 0 0

File: src/swc_nav_bringup/urdf/gkchair01_base_sim.urdf (robot description, URDF)
Before this commit: robot gk01, 1 links, 1 joints
Links:
- removed link livox_imu
Joints:
- removed joint livox_imu_joint

Commit message: 修改urdf模型

File: src/swc_nav_bringup/urdf/gkchair01_base.urdf (robot description, URDF)
Before this commit: robot gk01, 6 links, 5 joints
Links:
- added link astra_link; visual mesh filename=package://swc_nav_bringup/meshes/astra.STL scale=1.0 1.0 1.0
- link laser_link: geometry visual mesh filename=package://swc_nav_bringup/meshes/sls2.STL scale=1.0 1.0 1.0
- link livox_frame: geometry visual mesh filename=package://swc_nav_bringup/meshes/mid360.stl scale=0.0008 0.0008 0.0008
Joints:
- added joint astra_joint: type fixed, parent laser_link, child astra_link, origin xyz=0 0 0.03
- joint imu_joint: origin xyz=0 0 0.01 -> xyz=0 0 0
